Commit message: RVL path planning in Gazebo

File: ferit_ur5_ws/src/ur5_configs/ur5_robotiq3f_moveit_config/config/gazebo_ur5.urdf (robot description, URDF)
Before this commit: robot ur5, 25 links, 24 joints
Links:
- added link gripper_link
Joints:
- added joint gripper_joint: type fixed, parent tool0, child gripper_link, origin xyz=0 0 0.0535 rpy=-1.5707963267948966 -3.141592653589793 -1.5707963267948966
- joint finger_1_joint_1: origin xyz=0.020 0 0 rpy=0 -0.2 0 -> xyz=0.020 0 0 rpy=0 -0.2 0.065
- joint finger_2_joint_1: origin xyz=0.020 0 0 rpy=0 0.2 0 -> xyz=0.020 0 0 rpy=0 0.2 0.065
- joint finger_middle_joint_1: origin xyz=0.020 0 0 rpy=0 0 0 -> xyz=0.020 0 0 rpy=0 0 0.065

File: ferit_ur5_ws/src/ur5_configs/ur5_robotiq3f_moveit_config/config/gazebo_ur5_simplified.urdf (robot description, URDF)
Before this commit: robot ur5, 13 links, 12 joints
Joints:
- joint gripper_tool0_joint: origin xyz=0 0 0.1 rpy=0 0 -1.5707963267948966 -> xyz=0 0 0.115 rpy=0 0 -1.5707963267948966
