Commit message: TSR experiments for 1000 cabinets.

File: ferit_ur5_ws/cabinet_handle_test.urdf (robot description, URDF)
Before this commit: robot my_cabinet, 4 links, 3 joints
Links:
- link base_cabinet_link: geometry collision box size=0.018 0.39042122486281394 0.495788099859824; collision box size=0.4 0.018 0.495788099859824
- link door_link: geometry collision box size=0.018 0.34442122486281396 0.463788099859824; visual box size=0.018 0.34442122486281396 0.463788099859824
Joints:
- joint door_joint: origin xyz=0.191 -0.1400853789886163 0.0 rpy=0.000000 -0.000000 3.141593 -> xyz=0.191 -0.16221061243140697 0.0 rpy=0.000000 -0.000000 3.141593
- joint handle_joint: origin xyz=-0.028999999999999998 -0.25017075797723265 0.0 rpy=0.000000 -0.000000 3.141593 -> xyz=-0.028999999999999998 -0.29442122486281397 0.0 rpy=0.000000 -0.000000 3.141593
