Commit message: Debugged RVL; Debugged Moveit+Gazebo; Still making weird trajectories.

File: ferit_ur5_ws/cabinet.urdf (robot description, URDF)
Before this commit: robot my_cabinet, 3 links, 2 joints
Joints:
- joint door_joint: origin xyz=0.191 0.13999999999999999 0 rpy=0 0 3.141592653589793 -> xyz=0.191 0.13999999999999999 0 rpy=0 0 0

Commit message: finished simulation experiments & real experiment

File: ferit_ur5_ws/cabinet.urdf (robot description, URDF)
Before this commit: robot my_cabinet, 3 links, 2 joints
Links:
- link base_cabinet_link: geometry collision box size=0.018 0.3474355816880533 0.2949862502110655; collision box size=0.4 0.018 0.2949862502110655
- link door_link: geometry collision box size=0.018 0.3014355816880533 0.2629862502110655; visual box size=0.018 0.3014355816880533 0.2629862502110655
Joints:
- joint door_joint: origin xyz=0.141 -0.188 0 rpy=0 0 0 -> xyz=0.191 -0.14071779084402664 0 rpy=0 0 0

File: ferit_ur5_ws/src/ur5_configs/ur5_robotiq_ft_3f_moveit_config/config/gazebo_ur5_robotiq_ft_3f.urdf (robot description, URDF)
Before this commit: robot ur5_robotiq_ft_3f, 29 links, 28 joints
Links:
- link gripper_coupler: geometry collision cylinder length=0.028 radius=0.04; visual cylinder length=0.028 radius=0.04
Joints:
- joint ft_sensor_gripper_coupler_joint: origin xyz=0 0 -0.0065 rpy=3.141592653589793 0 0 -> xyz=0 0 -0.014 rpy=3.141592653589793 0 0
- joint gripper_coupler_robotiq_3f_joint: origin xyz=0 0 0.06 rpy=1.5707963267948966 0 -0.7853981633974483 -> xyz=0 0 0.068 rpy=1.5707963267948966 0 -0.7853981633974483

Commit message: Added ft sensor analysis; Added path_planning pkg

File: ferit_ur5_ws/cabinet.urdf (robot description, URDF)
Before this commit: robot my_cabinet, 3 links, 2 joints
Links:
- link base_cabinet_link: geometry collision box size=0.018 0.29617563489536053 0.6501201833097031; collision box size=0.4 0.018 0.6501201833097031
- link door_link: geometry collision box size=0.018 0.25017563489536054 0.6181201833097031; visual box size=0.018 0.25017563489536054 0.6181201833097031
Joints:
- joint door_joint: origin xyz=0.191 -0.14071779084402664 0 rpy=0 0 0 -> xyz=0.191 -0.11508781744768028 0 rpy=0 0 0

Commit message: Updated docker stuff and single-c

File: ferit_ur5_ws/cabinet.urdf (robot description, URDF)
Before this commit: robot my_cabinet, 3 links, 2 joints
Links:
- link base_cabinet_link: geometry collision box size=0.018 0.34519764983567797 0.3407406531608693; collision box size=0.3 0.018 0.3407406531608693
- link door_link: geometry collision box size=0.018 0.294197649835678 0.2947406531608693; visual box size=0.018 0.294197649835678 0.2947406531608693
Joints:
- joint door_joint: origin xyz=0.191 -0.1985 0.0 rpy=0.000000 -0.000000 3.141593 -> xyz=0.141 -0.147098824917839 0.0 rpy=0.000000 -0.000000 3.141593

Commit message: Some experiments

File: ferit_ur5_ws/cabinet.urdf (robot description, URDF)
Before this commit: robot my_cabinet, 4 links, 3 joints
Links:
- removed link handle_link
- link base_cabinet_link: geometry collision box size=0.018 0.32149466086151346 0.8103000519155183; collision box size=0.3 0.018 0.8103000519155183
- link door_link: geometry collision box size=0.018 0.27049466086151347 0.7643000519155183; visual box size=0.018 0.27049466086151347 0.7643000519155183
Joints:
- removed joint handle_joint
- joint door_joint: origin xyz=0.141 -0.16558663303811977 0.0 rpy=0.000000 -0.000000 3.141593 -> xyz=0.141 -0.13524733043075673 0.0 rpy=0.000000 -0.000000 3.141593

File: ferit_ur5_ws/cabinet_handle_test.urdf (robot description, URDF)
Before this commit: robot my_cabinet, 4 links, 3 joints
Links:
- link base_cabinet_link: geometry collision box size=0.018 0.26558210037472013 0.6938184815473808; collision box size=0.3 0.018 0.6938184815473808
- link door_link: geometry collision box size=0.018 0.21458210037472014 0.6478184815473808; visual box size=0.018 0.21458210037472014 0.6478184815473808
Joints:
- joint door_joint: origin xyz=0.141 -0.10458439207332615 0.0 rpy=0.000000 -0.000000 3.141593 -> xyz=0.141 -0.10729105018736007 0.0 rpy=0.000000 -0.000000 3.141593
- joint handle_joint: origin xyz=-0.028999999999999998 -0.1591687841466523 0.0 rpy=0.000000 -0.000000 3.141593 -> xyz=-0.028999999999999998 -0.16458210037472015 0.0 rpy=0.000000 -0.000000 3.141593

File: ferit_ur5_ws/src/ur5_configs/ur5_robotiq_ft_3f_moveit_config/config/gazebo_ur5_robotiq_ft_3f.urdf (robot description, URDF)
Before this commit: robot ur5_robotiq_ft_3f, 30 links, 29 joints
Links:
- removed link camera_link
Joints:
- removed joint camera_joint__
