Commit message: Adding Touch stuff to RVL; added force opening with ft and tactile to ferit_ur5_ws

File: ferit_ur5_ws/src/ur5_configs/fmauch_universal_robot/ur_description/urdf/ur5_robotiq_ft_3f.urdf.xacro (robot description, xacro)
@@ -73,4 +73,70 @@
       <child link="camera_link" />
   </joint>
+  <link name="gripper_power_plug">
+    <visual>
+      <origin xyz="0 0 0" rpy="0 0 0" />
+      <geometry>
+        <cylinder radius="0.008" length="0.048" />
+      </geometry>
+      <material name="Robotiq-Grey">
+          <color rgba="0.4 0.4 0.4 1.0"/>
+      </material>
+    </visual>
+    <collision>
+      <origin xyz="0 0 0" rpy="0 0 0"/>
+      <geometry>
+        <cylinder radius="0.008" length="0.048" />
+      </geometry>
+    </collision>
+    <inertial>
+      <origin xyz="0 0 0" rpy="0 0 0"/>
+      <mass value="0.1"/>
+      <inertia
+        ixx="0.0001"
+        ixy="0.0"
+        ixz="0.0"
+        iyy="0.0001"
+        iyz="0.0"
+        izz="0.0001"/>
+    </inertial>
+  </link>
+  <link name="gripper_ethernet_plug">
+    <visual>
+      <origin xyz="0 0 0" rpy="0 0 0" />
+      <geometry>
+        <cylinder radius="0.008" length="0.048" />
+      </geometry>
+      <material name="Robotiq-Grey">
+          <color rgba="0.4 0.4 0.4 1.0"/>
+      </material>
+    </visual>
+    <collision>
+      <origin xyz="0 0 0" rpy="0 0 0"/>
+      <geometry>
+        <cylinder radius="0.008" length="0.048" />
+      </geometry>
+    </collision>
+    <inertial>
+      <origin xyz="0 0 0" rpy="0 0 0"/>
+      <mass value="0.1"/>
+      <inertia
+        ixx="0.0001"
+        ixy="0.0"
+        ixz="0.0"
+        iyy="0.0001"
+        iyz="0.0"
+        izz="0.0001"/>
+    </inertial>
+  </link>
+  <joint name="gripper_power_plug_joint" type="fixed">
+    <origin xyz="0.09 -0.035 0.025" rpy="${pi/2} 0 0" />
+    <parent link="palm"/>
+    <child link="gripper_power_plug"/>
+  </joint>
+  <joint name="gripper_ethernet_plug_joint" type="fixed">
+    <origin xyz="0.09 -0.035 -0.025" rpy="${pi/2} 0 0" />
+    <parent link="palm"/>
+    <child link="gripper_ethernet_plug"/>
+  </joint>
   <link name="world" />
   <joint name="virtual_joint" type="fixed">
