Commit message: Updated robot URDF with new gripper and tactile sensor.

File: ferit_ur5_ws/src/ur5_configs/robotiq-noetic-devel/robotiq_ft_sensor/urdf/robotiq_ft300.urdf.xacro (robot description, xacro)
@@ -1,5 +1,5 @@
 <?xml version="1.0"?>
 <!-- Develped by: Daniel Ordonez 20.06.2019 - daniels.ordonez@gmail.com-->
-<robot xmlns:xacro="http://ros.org/wiki/xacro" name="robotiq_fts150">
+<robot xmlns:xacro="http://ros.org/wiki/xacro" name="robotiq_ft300">
     <!-- Macro function to instanciate URDF model of the FT300 force-torque sensor with mounting plate
         Example use:
@@ -62,5 +62,5 @@
         </link>
          <!-- Connect force sensor with mounting/coupling plate -->
-        <joint name="${prefix}ft300_mounting_plate" type="fixed">
+        <joint name="${prefix}ft300_mounting_plate_ft300_sensor_joint" type="fixed">
             <origin xyz="0 0 0.0415" rpy="0 ${pi} 0"/>
             <parent link="${prefix}ft300_mounting_plate" />
