Commit message: Fused multi-contact with Touch.

File: ferit_ur5_ws/src/ur5_configs/ur5_robotiq_ft_3f_moveit_config/config/gazebo_ur5_robotiq_ft_3f_new_mesh.urdf (robot description, URDF)
Before this commit: robot ur5_robotiq_ft_3f, 35 links, 34 joints
Joints:
- removed joint robotiq_3f_frame_to_AGS_palm_joint
- added joint AGS_wrist_to_AGS_palm_joint: type fixed, parent AGS_wrist, child AGS_palm, origin xyz=0 -0.04127 0 rpy=0 1.0432366 3.1415927
